File: PCB Files/TFTAudio.kicad_sch (KiCad schematic)
At the start: 55 parts, among them J2 Lipo 1S, J3 Display, J4 AudioJack3, J5 expansion, J6 USB_C_Receptacle_USB2.0_14P, Q1 BSS138, Q2 BSS138, Q3 DMG2301L, SW1 SW_SPST, SW2 RESET, U1 ESP32-WROVER-E, U2 CH340C, U3 MCP73831-2-OT, U4 AP2112K-3.3, U5 PCM5102A

Commit message: PCB Draft 5
Parts:
- SW2: footprint Button_Switch_THT:SW_Tactile_SKHH_Angled -> Button_Switch_SMD:SW_SPST_EVQP7C; LCSC C318884 -> C318884
Changed lines of the file:
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@@
 			)
 		)
-		(property "Footprint" "Button_Switch_THT:SW_Tactile_SKHH_Angled"
+		(property "Footprint" "Button_Switch_SMD:SW_SPST_EVQP7C"
 			(at 125.73 52.07 0)
 			(effects
@@
 			)
 		)
-		(property "LCSC" " C318884"
+		(property "LCSC" "C318884"
 			(at 130.81 52.07 90)
 			(effects

Commit message: Submitted PCB
Parts:
- C1, C15, C2, C23, C5, C7, C9: value 100n -> 100nF; LCSC C5137636 -> C14663
- C14, C22, C3, C4, C8: value 10u -> 10uF; LCSC C15850 -> C19702
- C16, C17: LCSC (none) -> C1604
- C18, C19, C25, C26: LCSC (none) -> C14663
- C20: LCSC (none) -> C19702
- C21, C24: LCSC (none) -> C23630
- C6: value 1u -> 10uF; LCSC C1592 -> C19702
- D1: LCSC C2296 -> C2286
- D2: LCSC C77335 -> C8598
- D3: LCSC C2297 -> C2286
- J2: LCSC C20422588 -> (none)
- J6: LCSC C165948 -> C165948
- Q1, Q2: value BSS138 -> AO3400A; LCSC C40912 -> C20917
- Q3: value DMG2301L -> AO3401A; footprint Package_TO_SOT_SMD:SOT-23 -> Package_TO_SOT_SMD; LCSC C7472914 -> C15127
- R1, R3: LCSC (none) -> C21190
- R10: value 220 -> 220R; LCSC (none) -> C22962
- R11: value 10k -> 10K; LCSC (none) -> C25804
- R2: value 2k -> 2.2k; LCSC (none) -> C4190
- R4, R5: LCSC (none) -> C23186
- R6, R7: LCSC (none) -> C23179
- R8: LCSC (none) -> C25804
- R9: value 100k -> 100K; LCSC (none) -> C25803
- SW2: LCSC C318884 -> C388883
Changed lines of the file:
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@@
 			)
 		)
-		(property "LCSC" " C165948"
+		(property "LCSC" "C165948"
 			(at 25.4 48.26 0)
 			(effects
@@
 			)
 		)
-		(property "LCSC" ""
+		(property "LCSC" "C21190"
 			(at 97.79 171.45 0)
 			(effects
@@
 			)
 		)
-		(property "LCSC" ""
+		(property "LCSC" "C14663"
 			(at 204.47 68.58 90)
 			(effects
@@
 			)
 		)
-		(property "Value" "100n"
+		(property "Value" "100nF"
 			(at 91.948 25.4 0)
 			(effects
@@
 			)
 		)
-		(property "LCSC" "C5137636"
+		(property "LCSC" "C14663"
 			(at 91.44 22.86 0)
 			(effects
@@
 			)
 		)
-		(property "Value" "10u"
+		(property "Value" "10uF"
 			(at 91.44 87.63 0)
 			(effects
@@
 			)
 		)
-		(property "LCSC" "C15850"
+		(property "LCSC" "C19702"
 			(at 90.17 85.09 0)
 			(effects
@@
 			)
 		)
-		(property "LCSC" ""
+		(property "LCSC" "C19702"
 			(at 204.47 78.74 90)
 			(effects
@@
 			)
 		)
-		(property "LCSC" ""
+		(property "LCSC" "C23630"
 			(at 212.09 45.72 90)
 			(effects
@@
 			)
 		)
-		(property "LCSC" " C2297"
+		(property "LCSC" "C2286"
 			(at 82.55 176.53 0)
 			(effects
@@
 			)
 		)
-		(property "LCSC" ""
+		(property "LCSC" "C23630"
 			(at 212.09 53.34 90)
 			(effects
@@
 			)
 		)
-		(property "Value" "BSS138"
+		(property "Value" "AO3400A"
 			(at 106.68 29.21 0)
 			(effects
@@
 			)
 		)
-		(property "LCSC" "C40912"
+		(property "LCSC" "C20917"
 			(at 111.76 35.56 0)
 			(effects
@@
 			)
 		)
-		(property "LCSC" "C2296"
+		(property "LCSC" "C2286"
 			(at 52.07 111.76 0)
 			(effects
@@
 			)
 		)
-		(property "LCSC" ""
+		(property "LCSC" "C14663"
 			(at 252.73 48.26 90)
 			(effects
@@
 			)
 		)
-		(property "Value" "10u"
+		(property "Value" "10uF"
 			(at 224.79 92.71 0)
 			(effects
@@
 			)
 		)
-		(property "LCSC" "C15850"
+		(property "LCSC" "C19702"
 			(at 223.52 90.17 0)
 			(effects
@@
 			)
 		)
-		(property "Value" "100n"
+		(property "Value" "100nF"
 			(at 234.95 92.71 0)
 			(effects
@@
 			)
 		)
-		(property "LCSC" "C5137636"
+		(property "LCSC" "C14663"
 			(at 233.68 90.17 0)
 			(effects
@@
 			)
 		)
-		(property "LCSC" ""
+		(property "LCSC" "C23179"
 			(at 190.5 58.42 0)
 			(effects
@@
 			)
 		)
-		(property "LCSC" ""
+		(property "LCSC" "C1604"
 			(at 179.07 64.77 90)
 			(effects
@@
 			)
 		)
-		(property "Value" "10k"
+		(property "Value" "10K"
 			(at 132.588 39.3121 0)
 			(effects
@@
 			)
 		)
-		(property "LCSC" ""
+		(property "LCSC" "C25804"
 			(at 130.81 38.1 0)
 			(effects
@@
 			)
 		)
-		(property "Value" "DMG2301L"
+		(property "Value" "AO3401A"
 			(at 69.85 155.575 0)
 			(effects
@@
 			)
 		)
-		(property "Footprint" "Package_TO_SOT_SMD:SOT-23"
+		(property "Footprint" "Package_TO_SOT_SMD"
 			(at 71.12 161.925 0)
 			(effects
@@
 			)
 		)
-		(property "LCSC" "C7472914"
+		(property "LCSC" "C15127"
 			(at 66.04 160.02 0)
 			(effects
@@
 			)
 		)
-		(property "Value" "100n"
+		(property "Value" "100nF"
 			(at 101.6 87.63 0)
 			(effects
@@
 			)
 		)
-		(property "LCSC" "C5137636"
+		(property "LCSC" "C14663"
 			(at 100.33 85.09 0)
 			(effects
@@
 			)
 		)
-		(property "Value" "BSS138"
+		(property "Value" "AO3400A"
 			(at 106.68 50.8 0)
 			(effects
@@
 			)
 		)
-		(property "LCSC" "C40912"
+		(property "LCSC" "C20917"
 			(at 111.76 55.88 0)
 			(effects
@@
 			)
 		)
+		(property "LCSC" "C14663"
+			(at 203.2 35.56 0)
+			(effects
+				(font
+					(size 1.27 1.27)
+				)
+				(hide yes)
+			)
+		)
 		(pin "1"
 		)
@@
 			)
 		)
-		(property "LCSC" ""
+		(property "LCSC" "C21190"
 			(at 52.07 120.65 0)
 			(effects
@@
 			)
 		)
-		(property "Value" "220"
+		(property "Value" "220R"
 			(at 77.47 187.325 0)
 			(effects
@@
 			)
 		)
-		(property "LCSC" ""
+		(property "LCSC" "C22962"
 			(at 82.55 185.42 0)
 			(effects
@@
 			)
 		)
-		(property "Value" "100n"
+		(property "Value" "100nF"
 			(at 121.92 55.88 0)
 			(effects
@@
 			)
 		)
-		(property "LCSC" "C5137636"
+		(property "LCSC" "C14663"
 			(at 120.65 53.34 0)
 			(effects
@@
 			)
 		)
-		(property "LCSC" ""
+		(property "LCSC" "C23186 "
 			(at 58.42 38.1 0)
 			(effects
@@
 			)
 		)
-		(property "Value" "2k"
+		(property "Value" "2.2k"
 			(at 27.178 138.3721 0)
 			(effects
@@
 			)
 		)
-		(property "LCSC" ""
+		(property "LCSC" "C4190"
 			(at 25.4 137.16 0)
 			(effects
@@
 			)
 		)
-		(property "Value" "100n"
+		(property "Value" "100nF"
 			(at 139.7 179.07 0)
 			(effects
@@
 			)
 		)
-		(property "LCSC" "C5137636"
+		(property "LCSC" "C14663"
 			(at 138.43 176.53 0)
 			(effects
@@
 			)
 		)
-		(property "LCSC" ""
+		(property "LCSC" "C23179"
 			(at 190.5 55.88 0)
 			(effects
@@
 			)
 		)
-		(property "LCSC" ""
+		(property "LCSC" "C1604"
 			(at 179.07 49.53 90)
 			(effects
@@
 			)
 		)
-		(property "Value" "100n"
+		(property "Value" "100nF"
 			(at 77.978 29.21 0)
 			(effects
@@
 			)
 		)
-		(property "LCSC" "C5137636"
+		(property "LCSC" "C14663"
 			(at 77.47 26.67 0)
 			(effects
@@
 			)
 		)
-		(property "LCSC" "C318884"
+		(property "LCSC" "C388883"
 			(at 130.81 52.07 90)
 			(effects
@@
 			)
 		)
-		(property "LCSC" "	C77335"
+		(property "LCSC" "	C8598 "
 			(at 58.42 168.91 0)
 			(effects
@@
 			)
 		)
-		(property "Value" "100k"
+		(property "Value" "100K"
 			(at 43.942 177.546 0)
 			(effects
@@
 			)
 		)
-		(property "LCSC" ""
+		(property "LCSC" "C25803"
 			(at 50.8 176.53 0)
 			(effects
@@
 			)
 		)
-		(property "LCSC" ""
+		(property "LCSC" "C23186 "
 			(at 58.42 40.64 0)
 			(effects
@@
 			)
 		)
-		(property "Value" "10u"
+		(property "Value" "10uF"
 			(at 259.08 133.35 0)
 			(effects
@@
 			)
 		)
-		(property "LCSC" "C15850"
+		(property "LCSC" "C19702"
 			(at 257.81 130.81 0)
 			(effects
@@
 			)
 		)
-		(property "LCSC" ""
+		(property "LCSC" "C25804"
 			(at 274.32 43.18 0)
 			(effects
@@
 			)
 		)
-		(property "LCSC" "C20422588"
+		(property "LCSC" ""
 			(at 63.5 125.73 0)
 			(effects
@@
 			)
 		)
-		(property "Value" "1u"
+		(property "Value" "10uF"
 			(at 71.12 29.21 0)
 			(effects
@@
 			)
 		)
-		(property "LCSC" "C1592"
+		(property "LCSC" "C19702"
 			(at 71.12 26.67 0)
 			(effects
@@
 			)
 		)
-		(property "Value" "100n"
+		(property "Value" "100nF"
 			(at 269.24 133.35 0)
 			(effects
@@
 			)
 		)
-		(property "LCSC" "C5137636"
+		(property "LCSC" "C14663"
 			(at 267.97 130.81 0)
 			(effects
@@
 			)
 		)
-		(property "LCSC" ""
+		(property "LCSC" "C14663"
 			(at 252.73 43.18 90)
 			(effects
@@
 			)
 		)
-		(property "Value" "10u"
+		(property "Value" "10uF"
 			(at 91.44 177.165 0)
 			(effects
@@
 			)
 		)
-		(property "LCSC" "C15850"
+		(property "LCSC" "C19702"
 			(at 90.17 175.26 0)
 			(effects
@@
 			)
 		)
-		(property "Value" "10u"
+		(property "Value" "10uF"
 			(at 129.54 179.07 0)
 			(effects
@@
 			)
 		)
-		(property "LCSC" "C15850"
+		(property "LCSC" "C19702"
 			(at 128.27 176.53 0)
 			(effects

Commit message: production
Parts:
- D1: LCSC C2286 -> C84256
- D2: LCSC C8598 -> C8598
- D3: LCSC C2286 -> C2296
- H1, H2, H3, H4: now in the parts list
- J4: LCSC (none) -> C20182914
- U4: LCSC C51118 -> C51118
Changed lines of the file:
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@@
 		(unit 1)
 		(exclude_from_sim no)
-		(in_bom no)
+		(in_bom yes)
 		(on_board yes)
 		(dnp no)
@@
 			)
 		)
-		(property "LCSC" "C2286"
+		(property "LCSC" "C2296"
 			(at 82.55 176.53 0)
 			(effects
@@
 			)
 		)
-		(property "LCSC" "C2286"
+		(property "LCSC" "C84256"
 			(at 52.07 111.76 0)
 			(effects
@@
 		(unit 1)
 		(exclude_from_sim no)
-		(in_bom no)
+		(in_bom yes)
 		(on_board yes)
 		(dnp no)
@@
 			)
 		)
+		(property "LCSC" "C20182914 "
+			(at 158.75 49.53 90)
+			(effects
+				(font
+					(size 1.27 1.27)
+				)
+				(hide yes)
+			)
+		)
 		(pin "T"
 		)
@@
 		(unit 1)
 		(exclude_from_sim no)
-		(in_bom no)
+		(in_bom yes)
 		(on_board yes)
 		(dnp no)
@@
 			)
 		)
-		(property "LCSC" "	C8598 "
+		(property "LCSC" "C8598 "
 			(at 58.42 168.91 0)
 			(effects
@@
 		(unit 1)
 		(exclude_from_sim no)
-		(in_bom no)
+		(in_bom yes)
 		(on_board yes)
 		(dnp no)
@@
 			)
 		)
-		(property "LCSC" "	C51118"
+		(property "LCSC" "C51118"
 			(at 113.03 171.45 0)
 			(effects
