File: PCB Files/TFTAudio.kicad_pcb (KiCad board)
At the start: 2 copper layers, 108 x 60.9 mm, 55 parts, among them J2 Lipo 1S, J3 Display, J4 AudioJack3, J5 expansion, J6 USB_C_Receptacle_USB2.0_14P, Q1 AO3400A, Q2 AO3400A, Q3 AO3401A, SW1 SW_SPST, SW2 RESET, U1 ESP32-WROVER-E, U2 CH340C, U3 MCP73831-2-OT, U4 AP2112K-3.3, U5 PCM5102A

Commit message: Post submit tweaks
Parts:
- moved R8 0.98 mm to (98.9, 52.2), turned to 0 degrees
Routing:
- net GND: track 478.8 -> 111.0 mm, vias 6 -> 24
- net Net-(U5-XSMT): track 9.75 -> 4.83 mm, vias 2 -> 0
- net +3.3V: track 239.4 -> 237.7 mm
- net +5V: track 118.9 -> 119.9 mm

Commit message: production
Parts:
- moved SW2 0.72 mm to (59.1, 76.3), turned to 0 degrees
Routing:
- net /EN: track 77.0 -> 82.7 mm
- net GND: track 111.0 -> 116.2 mm, vias 24 -> 25
- net +5V: track 119.9 -> 124.6 mm
- net Net-(U3-STAT): track 18.3 -> 21.5 mm
- net /SWIN: track 27.5 -> 29.3 mm
- net /LCD_CS: track 47.1 -> 48.5 mm
- net +3.3V: track 237.7 -> 238.9 mm
- net Net-(J2-Pin_1): track 80.0 -> 81.2 mm
- net /CTP_SCL: track 130.1 -> 129.2 mm
- net /SCK: track 20.8 -> 20.0 mm
- net /RX: track 46.1 -> 46.9 mm
- net /GPIO19: track 108.5 -> 109.2 mm
- net /TX: track 45.6 -> 46.3 mm

Commit message: Production PCB v1.1
Other:
- board text added: "Alan Trundle ESP32 WROVER Audio DAC Board V1.1 16MB Flash / 8MB PSRAM 14/12/2025"
- board text removed: "Alan Trundle ESP32 WROVER Audio DAC Board V1.0 8MB Flash / 8MB PSRAM 14/12/2025"
Changed lines of the file:
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@@
 		)
 	)
-	(gr_text "Alan Trundle\nESP32 WROVER Audio DAC Board V1.0\n8MB Flash / 8MB PSRAM\n14/12/2025"
+	(gr_text "Alan Trundle\nESP32 WROVER Audio DAC Board V1.1\n16MB Flash / 8MB PSRAM\n14/12/2025"
 		(at 76.03 77.79 0)
 		(layer "F.SilkS")
